File: UccMicroDuino/UccMicroDuino.kicad_sch (KiCad schematic)
At the start: 8 parts, among them J2 Conn_01x10_Socket, J2 USB_A, U2 ATtiny85-20S

Commit message: Diseño de circuito en KiCad finalizado
Parts:
- added D4: LED GREEN, symbol Device:LED
- added D5: 3.6 V 1/2 W, Diode_SMD:D_SOD-123, symbol Device:D_Zener
- added R2: 300 omhs 5% 1/8w, symbol Device:R
- added R3, R4: 68 omhs 5% 1/8w, symbol Device:R
- D2: renamed from D1; value D_Zener -> 3.6 V 1/2 W
- R1: value R -> 1.5 omhs 5% 1/8w
- renumbered D5 to D1, J2 to J1, U2 to U1
Connections:
- net +5V: now also U1.8 (VCC)
- net GND: now also D2.2 (A), J1.2 (Pin_2), J2.4 (GND), D5.2 (A), R2.2
- net at R1.2: now also D2.1 (K), J2.2 (D-), R4.1
- net at U1.1 (~{RESET}/PB5): now also J1.9 (Pin_9)
- net at U1.2 (XTAL1/PB3): now also J1.7 (Pin_7), R4.2
- net at U1.3 (XTAL2/PB4): now also J1.8 (Pin_8), R3.2
- net at U1.5 (AREF/PB0): now also J1.4 (Pin_4)
- net at U1.6 (PB1): now also J1.5 (Pin_5), D4.2 (A)
- net at U1.7 (PB2): now also J1.6 (Pin_6)
- net at J2.1 (VBUS): now also D1.2 (A)
- net at J2.3 (D+): now also D5.1 (K), R3.1
- new net: D4.1 (K), R2.1
- no-connect marks 0 -> 2
Other:
- moved on the sheet: J1, U1
