File: UccMicroDuino/UccMicroDuino.kicad_sch (KiCad schematic)
At the start: 13 parts, among them J1 Conn_01x10_Socket, J2 USB_A, U1 ATtiny85-20S

Commit message: arreglo
Parts:
- added R5: 300 omhs 5% 1/8w, symbol Device:R
- C1: value C -> 0.1u
- D3: value LED -> LED RED
- D4: footprint (none) -> ledSmd:ledSMD
- R2, R3, R4: footprint (none) -> Resistor_SMD:R_0805_2012Metric_Pad1.20x1.40mm_HandSolder
- U1: footprint Package_SO:SOIC-8W_5.3x5.3mm_P1.27mm -> Package_SO:SOIC-8_5.3x5.3mm_P1.27mm
Connections:
- net +5V: now also C1.1, D3.2 (A), J1.1 (Pin_1)
- net GND: now also C1.2, U1.4 (GND), R5.2
- net at D3.1 (K): now also R5.1
Other:
- note added: "DC Power"
- note added: "Power Led"
- moved on the sheet: D3

Commit message: clase 5 de mayo
Parts:
- R5: footprint (none) -> Resistor_SMD:R_0805_2012Metric_Pad1.20x1.40mm_HandSolder
Changed lines of the file:
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@@
 			)
 		)
-		(property "Footprint" ""
+		(property "Footprint" "Resistor_SMD:R_0805_2012Metric_Pad1.20x1.40mm_HandSolder"
 			(at 256.032 87.63 90)
 			(effects
